File: workspace/systemMonitorLab/hardware/PcbSistemaAmbienteLab/PcbSistemaAmbienteLab.kicad_sch (KiCad schematic)
At the start: 2 parts

Commit message: Esquemativo v1.0 y PCB v1.0
Parts:
- removed U?: DHT11, Sensor:Aosong_DHT11_5.5x12.0_P2.54mm, symbol Sensor:DHT11
- added J1, J2: Conn_01x01_Male, Connector_Pin:Pin_D1.0mm_L10.0mm, symbol Connector:Conn_01x01_Male
- added R1: 5K6, Resistor_THT:R_Axial_DIN0411_L9.9mm_D3.6mm_P12.70mm_Horizontal, symbol Device:R
- added U1: DHT22, Sensor:Aosong_DHT11_5.5x12.0_P2.54mm, symbol New_Library:DHT22
- added U2: AHT10, Connector_PinHeader_2.54mm:PinHeader_1x04_P2.54mm_Vertical, symbol New_Library:AHT10
- added U3: Bmp280Module, Connector_PinHeader_2.54mm:PinHeader_1x06_P2.54mm_Vertical, symbol New_Library:Bmp280Module
- U4: renamed from U?; footprint Module:Adafruit_Feather_32u4_FONA -> NodeMCU_Module:ES8266
Connections:
- net +5V: now also U4.15 (Vin), J1.1 (Pin_1), R1.1
- net GND: now also U4.14 (GND), U4.16 (GND), U4.24 (GND), J2.1 (Pin_1), U1.4 (GND), U2.2 (GND), U3.2 (GND), U3.6 (SDO)
- net 3V3: now reaches U4.11 (3V3)
- net 3V3: now also U4.17 (3V3), U4.25 (3V3), U1.1 (VCC), U2.1 (VCC), U3.1 (VCC), U3.5 (CSB)
- net at U4.23 (IO14/SCK): now also U2.4 (SDA), U3.4 (SDA)
- net at U4.26 (IO2): now also U2.3 (SCL), U3.3 (SCL)
- net at U4.28 (SDA/IO4): now also R1.2, U1.2 (IO)
- no-connect marks 0 -> 20
Other:
- company: (none) -> Servicio Meteorológico Nacional (SMN)
- title: (none) -> Sensores de temperatura, humedad y presión

Commit message: Esquematico y PCB para sistema de monitoreo v1.1
Parts:
- R1: footprint Resistor_THT:R_Axial_DIN0411_L9.9mm_D3.6mm_P12.70mm_Horizontal -> Resistor_THT:R_Axial_DIN0207_L6.3mm_D2.5mm_P10.16mm_Horizontal
- U4: footprint NodeMCU_Module:ES8266 -> NodeMCU_Module:ESP8266
Connections:
- net +5V: no longer R1.1
- net 3V3: now also R1.1; no longer U4.17 (3V3), U4.25 (3V3)
- net GND: now also U4.10 (GND); no longer U4.14 (GND), U4.16 (GND), U4.24 (GND)
- no-connect marks 20 -> 24

Commit message: subo v1.2 del PCB del sistema de monitoreo ambiente, esta versión se utilizara para calibrar el sensor AHT10 vs DHT22
Parts:
- R1: footprint Resistor_THT:R_Axial_DIN0207_L6.3mm_D2.5mm_P10.16mm_Horizontal -> Resistor_THT:R_Axial_DIN0207_L6.3mm_D2.5mm_P15.24mm_Horizontal
Connections:
- net GND: now also U4.17 (GND), U4.24 (GND)
- no-connect marks 24 -> 22
Changed lines of the file:
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@@
   (no_connect (at 168.402 77.978))
   (no_connect (at 168.402 109.728))
-  (no_connect (at 168.402 81.788))
   (no_connect (at 143.002 81.788))
   (no_connect (at 143.002 113.538))
@@
   (no_connect (at 168.402 90.678))
   (no_connect (at 168.402 69.088))
-  (no_connect (at 168.402 113.538))
   (no_connect (at 143.002 77.978))
   (no_connect (at 143.002 86.868))
@@
     )
     (property "Datasheet" "" (id 3) (at 211.074 129.794 0)
+      (effects (font (size 1.27 1.27)) hide)
+    )
+    (pin "1")
+  )
+  (symbol (lib_id "power:GND") (at 168.402 113.538 90) (unit 1)
+    (in_bom yes) (on_board yes) (fields_autoplaced)
+    (property "Reference" "#PWR?" (id 0) (at 174.752 113.538 0)
+      (effects (font (size 1.27 1.27)) hide)
+    )
+    (property "Value" "GND" (id 1) (at 172.466 113.5379 90)
+      (effects (font (size 1.27 1.27)) (justify right))
+    )
+    (property "Footprint" "" (id 2) (at 168.402 113.538 0)
+      (effects (font (size 1.27 1.27)) hide)
+    )
+    (property "Datasheet" "" (id 3) (at 168.402 113.538 0)
       (effects (font (size 1.27 1.27)) hide)
     )
@@
     (pin "4")
   )
+  (symbol (lib_id "power:GND") (at 168.402 81.788 90) (unit 1)
+    (in_bom yes) (on_board yes) (fields_autoplaced)
+    (property "Reference" "#PWR0103" (id 0) (at 174.752 81.788 0)
+      (effects (font (size 1.27 1.27)) hide)
+    )
+    (property "Value" "GND" (id 1) (at 172.593 81.7879 90)
+      (effects (font (size 1.27 1.27)) (justify right))
+    )
+    (property "Footprint" "" (id 2) (at 168.402 81.788 0)
+      (effects (font (size 1.27 1.27)) hide)
+    )
+    (property "Datasheet" "" (id 3) (at 168.402 81.788 0)
+      (effects (font (size 1.27 1.27)) hide)
+    )
+    (pin "1")
+  )
   (symbol (lib_id "Connector:Conn_01x01_Male") (at 254.254 33.274 180) (unit 1)
     (in_bom yes) (on_board yes) (fields_autoplaced)
@@
       (effects (font (size 1.27 1.27)) (justify left))
     )
-    (property "Footprint" "Resistor_THT:R_Axial_DIN0207_L6.3mm_D2.5mm_P10.16mm_Horizontal" (id 2) (at 187.325 43.18 90)
+    (property "Footprint" "Resistor_THT:R_Axial_DIN0207_L6.3mm_D2.5mm_P15.24mm_Horizontal" (id 2) (at 187.325 43.18 90)
       (effects (font (size 1.27 1.27)) hide)
     )
@@
       (reference "#PWR0102") (unit 1) (value "GND") (footprint "")
     )
+    (path "/a095de42-9687-4a0d-93b3-dc0b87f328f2"
+      (reference "#PWR0103") (unit 1) (value "GND") (footprint "")
+    )
     (path "/17335677-c6e0-40da-858c-7f570741789f"
       (reference "#PWR0104") (unit 1) (value "GND") (footprint "")
@@
       (reference "#PWR0109") (unit 1) (value "GND") (footprint "")
     )
+    (path "/186b7442-f1d8-4f2b-a24e-5cad9ec9a5c2"
+      (reference "#PWR?") (unit 1) (value "GND") (footprint "")
+    )
     (path "/056d7cd6-72a4-409b-84e3-a39aef2e8b6b"
       (reference "J1") (unit 1) (value "Conn_01x01_Male") (footprint "Connector_Pin:Pin_D1.0mm_L10.0mm")
@@
     )
     (path "/fb82c059-0a4d-4eab-ba6b-b1bb9f915050"
-      (reference "R1") (unit 1) (value "5K6") (footprint "Resistor_THT:R_Axial_DIN0207_L6.3mm_D2.5mm_P10.16mm_Horizontal")
+      (reference "R1") (unit 1) (value "5K6") (footprint "Resistor_THT:R_Axial_DIN0207_L6.3mm_D2.5mm_P15.24mm_Horizontal")
     )
     (path "/da8e9a8f-ad31-4f1a-bc50-16f63337dd07"
