File: workspace/systemMonitorLab/hardware/NodoAmbienteSMN/NodoV2/shield_base.kicad_sch (KiCad schematic)
At the start: 5 parts, among them J1 DHT22, J2 BMP280, J3 Jack-DC, U1 NodeMcuEsp8266

Commit message: Se agregan leds de estado con sus respectivos conectores y se agrega en el codigo la configuracion de los GPIO para usar estos leds como indicadores de envio de datos, conexion con el servidor Web Socket y conectividad wifi
Parts:
- added J6: Molex_MainBoard_Led_Status, Connector_PinHeader_2.54mm:PinHeader_1x05_P2.54mm_Horizontal, symbol Connector:Conn_01x05_Male
- added Q1, Q2, Q3, Q4: Q_NPN_BEC, Package_TO_SOT_SMD:SOT-23, symbol Device:Q_NPN_BEC
- added R2, R4, R8, R9: 1k, Resistor_SMD:R_1206_3216Metric, symbol Device:R
- added R3, R5, R6, R7: 39, Resistor_SMD:R_1206_3216Metric, symbol Device:R
- J1: value DHT22 -> Molex_MainBoard_DHT22; footprint (none) -> Connector_PinHeader_2.54mm:PinHeader_1x04_P2.54mm_Horizontal
- J2: value BMP280 -> Molex_MainBoard_BMP280; footprint (none) -> Connector_PinHeader_2.54mm:PinHeader_1x04_P2.54mm_Horizontal
- J3: footprint (none) -> Connector_BarrelJack:BarrelJack_GCT_DCJ200-10-A_Horizontal
- R1: footprint Resistor_THT:R_Axial_DIN0207_L6.3mm_D2.5mm_P15.24mm_Horizontal -> Resistor_SMD:R_1206_3216Metric
- U1: footprint NodeMCU_Module:ESP8266 -> NodeMCU_Module:ESP8266_v3
Connections:
- net +5V: now also J3.1, Q1.3 (C), Q2.3 (C), Q3.3 (C), Q4.3 (C); no longer J3.2
- net GND: now also J3.2, J6.1 (Pin_1); no longer J3.1
- net LED_GREEN: now reaches U1.20 (IO15)
- net LED_GREEN: now also R9.1
- net LED_DUAL_GREEN: now reaches U1.21 (IO13/MOSI)
- net LED_DUAL_GREEN: now also R8.1
- net LED_DUAL_RED: now reaches U1.22 (IO12/MISO)
- net LED_DUAL_RED: now also R4.1
- net LED_YELLOW: now reaches U1.29 (SCL/IO5)
- net LED_YELLOW: now also R2.1
- new net: J6.2 (Pin_2), R3.2
- new net: J6.3 (Pin_3), R5.2
- new net: J6.4 (Pin_4), R6.2
- new net: J6.5 (Pin_5), R7.2
- new net: Q3.1 (B), R8.2
- new net: Q4.1 (B), R9.2
- new net: Q1.2 (E), R3.1
- new net: Q4.2 (E), R7.1
- new net: Q3.2 (E), R6.1
- new net: Q2.1 (B), R4.2
- new net: Q2.2 (E), R5.1
- new net: Q1.1 (B), R2.2
- no-connect marks 23 -> 19
Other:
- moved on the sheet: J1, J2, R1, U1
